Commit message: tarea 4 - 1

File: robot_description/urdf/robot.xacro (robot description, xacro)
@@ -103,5 +103,5 @@
     <link name="ur_to_robotiq_adapter">
         <visual>
-            <origin xyz="0.000 0.000 1.359" rpy="0.000 0.000 0.000"/>
+            <origin xyz="0.000 0.000 -0.04" rpy="3.1416 0.000 0.000"/>
             <geometry>
                 <mesh filename="package://robot_description/meshes/visual/ur_to_robotiq_adapter.dae"/>
@@ -109,5 +109,5 @@
         </visual>
         <collision>
-            <origin xyz="0.000 0.000 1.359" rpy="0.000 0.000 0.000"/>
+            <origin xyz="0.000 0.000 -0.04" rpy="3.1416 0.000 0.000"/>
             <geometry>
                 <mesh filename="package://robot_description/meshes/collision/ur_to_robotiq_adapter.stl"/>
@@ -117,5 +117,5 @@
     <link name="robotiq_base">
         <visual>
-            <origin xyz="0.000 0.000 1.359" rpy="0.000 0.000 0.000"/>
+            <origin xyz="0.000 0.000 -0.055" rpy="3.1416 0.000 0.000"/>
             <geometry>
                 <mesh filename="package://robot_description/meshes/visual/robotiq_base.dae"/>
@@ -123,5 +123,5 @@
         </visual>
         <collision>
-            <origin xyz="0.000 0.000 1.359" rpy="0.000 0.000 0.000"/>
+            <origin xyz="0.000 0.000 -0.55" rpy="3.1416 0.000 0.000"/>
             <geometry>
                 <mesh filename="package://robot_description/meshes/collision/robotiq_base.stl"/>
